File: Hardware/lifepo4ups.kicad_sch (KiCad schematic)
At the start: 129 parts, among them J1 VBAT, J10 SWD, J11 BOOT, J2 VBAT_JST, J3 USB_C_Receptacle_USB2.0, J4 VIN, J5 VOUT, J6 UART1, J7 UART2, J8 Pogo pins, J9 VCC, Q1 Q_PMOS_GDS, Q2 Q_PMOS_GDS, Q3 BATFET, Q4 Q_NMOS_GDS, Q5 Q_NMOS_GDS, SW1 RST, U1 MAX17260SETD+T, U2 BQ24630RGER, U3 AP22966DC8-7, U4 TPS61230DRC, U5 STM32F030C8Tx, U6 INA219AxD, U7 NCP1117-3.3_SOT223, Y1 Crystal_Small

Commit message: Update schematic
Parts:
- removed C43, C45: DNP, symbol Local:C_Polarized_Small
- removed JP3: H_GND, Jumper:SolderJumper-2_P1.3mm_Open_RoundedPad1.0x1.5mm, symbol Jumper:SolderJumper_2_Open
- removed Q4, Q5: Q_NMOS_GDS, symbol Device:Q_NMOS_GDS
- added C22: 100n 10%, Capacitor_SMD:C_0805_2012Metric, symbol Local:C_Small
- added Q4: TDM3412, libraries:DFN3x3E-8_EP2_S, symbol Local:TDM3412
- BT1: footprint Battery:BatteryHolder_Keystone_1042_1x18650 -> libraries:BatteryHolder_Keystone_1043_1x18650
- C1, C2: value ? 25V -> ? 20% 25V; footprint (none) -> Capacitor_SMD:C_0805_2012Metric
- C10, C9: value 100n -> 100n 10%
- C11: value 470n -> 470n 10%; footprint (none) -> Capacitor_SMD:C_0805_2012Metric; Type (none) -> MLCC X5R
- C12, C13: value 1u -> 1u 10%
- C14, C15, C16: value 100n -> 100n 10%; footprint (none) -> Capacitor_SMD:C_0805_2012Metric; Type MLCC -> MLCC X7R
- C17: value 1u -> 1u 10%; footprint (none) -> Capacitor_SMD:C_0805_2012Metric; Type MLCC -> MLCC X7R
- C18: footprint (none) -> Capacitor_SMD:C_0805_2012Metric
- C19: value C_Small -> ? 10%; Type MLCC -> MLCC X7R
- C20: value C_SMALL -> 22u 20%
- C21: value 4u7 -> 4u7 10%; footprint (none) -> Capacitor_SMD:C_0805_2012Metric; Type (none) -> MLCC X5R
- C23: renamed from C22; value 100n -> 100n 10%
- C24: renamed from C23; value 100n -> 100n 10%
- C25: renamed from C24; value 10n -> 10n 10%; Type MLCC -> MLCC X5R
- C26: renamed from C25; value 1u -> 1u 10%
- C28: renamed from C27; value ???? -> ??; footprint (none) -> Capacitor_SMD:C_0805_2012Metric; Type (none) -> MLCC X5R
- C3, C5: value C_Small -> OPT 100n 10%; footprint (none) -> Capacitor_SMD:C_0805_2012Metric; Type (none) -> MLCC X7R
- C30: renamed from C29; value 1u -> 1u 20%; Type MLCC -> MLCC X5R
- C31: renamed from C30; value 1u -> 1u 20%; Type MLCC -> MLCC X5R
- C35: renamed from C34; footprint (none) -> Capacitor_SMD:C_0805_2012Metric
- C36: renamed from C35; footprint (none) -> Capacitor_SMD:C_0805_2012Metric
- C37: renamed from C36; value ?? 25V -> 5% 25V
- C38: renamed from C37; value ?? 25V -> 5% 25V
- C39: renamed from C38; value 100n -> 100n 10%; footprint (none) -> Capacitor_SMD:C_0805_2012Metric; Type MLCC -> MLCC X5R
- C4: value C_Small -> 10u 20%; footprint (none) -> Capacitor_SMD:C_0805_2012Metric
- C41: renamed from C40; value 100n -> 100n 10%
- C42: renamed from C41; value 10u -> 10u 20%; Type MLCC -> MLCC X5R
- C43: renamed from C42; footprint (none) -> Capacitor_Tantalum_SMD:CP_EIA-2012-15_AVX-P
- C45: renamed from C44; footprint (none) -> Capacitor_Tantalum_SMD:CP_EIA-2012-15_AVX-P
- C47: renamed from C46; value 10u -> 10u 20%; Type MLCC -> MLCC X5R
- C7: renamed from C8; value 100n -> 100n 10%; footprint (none) -> Capacitor_SMD:C_0805_2012Metric; Type MLCC -> MLCC X7R
- C8: renamed from C6; value C_Small -> 10u 10%; footprint (none) -> Capacitor_SMD:C_0805_2012Metric
- L1: value L_Small -> 15u 20%; footprint (none) -> libraries:L_1050
- L2: value L_Small -> 1u 20%; footprint (none) -> libraries:L_7030
- Q3: footprint (none) -> Package_TO_SOT_SMD:SOT-23
- R32: value ?? 1% -> 402k 1%
- R36: value ?? 1% -> 100k 1%
- R42: value R_Small -> ??
- R43: value R_Small -> 10k
- renumbered C26 to C27, C28 to C29, C31 to C32, C32 to C33, C33 to C34, C39 to C40, C7 to C6
Connections:
- net +3V3: now also C21.1, C23.2, C24.2, C22.2; no longer C21.2, C23.1, C24.1
- net +5V: now also C28.2; no longer C28.1
- net GND: now also C21.2, C23.1, C24.1, C28.1, C8.2, C22.1, Q4.5 (S2), Q4.6 (S2), Q4.7 (S2); no longer C21.1, C23.2, C24.2, C28.2, C8.1
- net HIDRV: now also Q4.1 (G1)
- net LODRV: now also Q4.8 (G2)
- net VCC: now also C8.1, Q4.2 (D1), Q4.3 (D1), Q4.4 (D1); no longer C8.2
- net PH: now reaches C14.2, L1.1, U2.20 (PH)
- net PH: now also Q4.9 (S1/D2)
- removed net GND1: H1.1, H2.1, H3.1, H4.1
- no-connect marks 16 -> 34
Other:
- note added: "C_{IN} 15u 20% X7R can also be used"
- note added: "C_{OUT} Maybe 10-15u for good loop stability"
- moved on the sheet: C21, C23, C24, C28, C8
