File: Hardware/lifepo4ups.kicad_pcb (KiCad board)
At the start: 2 copper layers, 85 x 56 mm, 0 parts

Commit message: Start layout
Parts:
- added BT1: 18650, libraries:BatteryHolder_Keystone_1043_1x18650, B.Cu at (126.4, 78.0)
- added C1: ? 20% 25V, Capacitor_SMD:C_0805_2012Metric, F.Cu at (144.0, 79.0)
- added C10: 100n 10%, Capacitor_SMD:C_0805_2012Metric, F.Cu at (84.0, 94.0)
- added C11: 470n 10%, Capacitor_SMD:C_0805_2012Metric, F.Cu at (57.0, 65.0)
- added C12: 1u 10%, Capacitor_SMD:C_0805_2012Metric, F.Cu at (72.5, 89.0)
- added C13: 1u 10%, Capacitor_SMD:C_0805_2012Metric, F.Cu at (82.0, 89.0)
- added C14: 100n 10%, Capacitor_SMD:C_0805_2012Metric, F.Cu at (73.0, 86.0)
- added C15: 100n 10%, Capacitor_SMD:C_0805_2012Metric, F.Cu at (84.0, 89.0)
- added C16: 100n 10%, Capacitor_SMD:C_0805_2012Metric, F.Cu at (82.0, 86.0)
- added C17: 1u 10%, Capacitor_SMD:C_0805_2012Metric, F.Cu at (72.0, 82.0)
- added C18: 150n 5% 25V, Capacitor_SMD:C_0805_2012Metric, F.Cu at (88.0, 92.0)
- added C19: ? 10%, Capacitor_SMD:C_0805_2012Metric, F.Cu at (20.0, 131.0)
- added C2: ? 20% 25V, Capacitor_SMD:C_0805_2012Metric, F.Cu at (144.0, 81.0)
- added C20: 22u 20%, Capacitor_SMD:C_0805_2012Metric, F.Cu at (83.0, 79.0)
- added C21: 4u7 10%, Capacitor_SMD:C_0805_2012Metric, F.Cu at (115.0, 96.0)
- added C22: 100n 10%, Capacitor_SMD:C_0805_2012Metric, F.Cu at (103.0, 88.0)
- added C23: 100n 10%, Capacitor_SMD:C_0805_2012Metric, F.Cu at (117.0, 96.0)
- added C24: 100n 10%, Capacitor_SMD:C_0805_2012Metric, F.Cu at (109.0, 83.0)
- added C25: 10n 10%, Capacitor_SMD:C_0805_2012Metric, F.Cu at (103.0, 92.0)
- added C26: 1u 10%, Capacitor_SMD:C_0805_2012Metric, F.Cu at (100.0, 92.0)
- added C28: ??, Capacitor_SMD:C_0805_2012Metric, F.Cu at (73.0, 73.0)
- added C29: 100n 10%, Capacitor_SMD:C_0805_2012Metric, F.Cu at (111.0, 63.0)
- added C3: OPT 100n 10%, Capacitor_SMD:C_0805_2012Metric, F.Cu at (24.5, 77.0)
- added C30: 1u 20%, Capacitor_SMD:C_0805_2012Metric, F.Cu at (102.0, 64.0)
- added C31: 1u 20%, Capacitor_SMD:C_0805_2012Metric, F.Cu at (110.0, 67.0)
- added C33: DNP, Capacitor_SMD:C_0805_2012Metric, F.Cu at (75.0, 82.0)
- added C34: 100n 10%, Capacitor_SMD:C_0805_2012Metric, F.Cu at (102.0, 59.0)
- added C35: ?? 5%, Capacitor_SMD:C_0805_2012Metric, F.Cu at (116.0, 77.0)
- added C36: ?? 5%, Capacitor_SMD:C_0805_2012Metric, F.Cu at (116.0, 73.0)
- added C37: 5% 25V, Capacitor_SMD:C_0805_2012Metric, F.Cu at (118.0, 63.0)
- added C38: 5% 25V, Capacitor_SMD:C_0805_2012Metric, F.Cu at (115.0, 63.0)
- added C39: 100n 10%, Capacitor_SMD:C_0805_2012Metric, F.Cu at (82.0, 69.0)
- added C4: 10u 20%, Capacitor_SMD:C_0805_2012Metric, F.Cu at (30.5, 77.0)
- added C40: DNP, Capacitor_SMD:C_0805_2012Metric, F.Cu at (92.0, 69.0)
- added C41: 100n 10%, Capacitor_SMD:C_0805_2012Metric, F.Cu at (90.0, 97.0)
- added C42: 10u 20%, Capacitor_SMD:C_0805_2012Metric, F.Cu at (97.0, 79.0)
- added C43: DNP, Capacitor_Tantalum_SMD:CP_EIA-2012-15_AVX-P, F.Cu at (95.0, 79.0)
- added C45: DNP, Capacitor_Tantalum_SMD:CP_EIA-2012-15_AVX-P, F.Cu at (110.0, 77.0)
- added C47: 10u 20%, Capacitor_SMD:C_0805_2012Metric, F.Cu at (108.0, 77.0)
- added C5: OPT 100n 10%, Capacitor_SMD:C_0805_2012Metric, F.Cu at (79.0, 129.0)
- added C7: 100n 10%, Capacitor_SMD:C_0805_2012Metric, F.Cu at (84.0, 92.0)
- added C8: 10u 10%, Capacitor_SMD:C_0805_2012Metric, F.Cu at (68.5, 93.0)
- added C9: 100n 10%, Capacitor_SMD:C_0805_2012Metric, F.Cu at (65.0, 65.0)
- added D2: LED_Small, LED_SMD:LED_0805_2012Metric, F.Cu at (53.5, 94.0)
- added D3: LED_Small, LED_SMD:LED_0805_2012Metric, F.Cu at (53.5, 90.0)
- added D4: LED_Small, LED_SMD:LED_0805_2012Metric, F.Cu at (53.5, 86.0)
- added H1: M2.5, MountingHole:MountingHole_2.7mm_M2.5_Pad, F.Cu at (111.5, 102.5)
- added H2: M2.5, MountingHole:MountingHole_2.7mm_M2.5_Pad, F.Cu at (111.5, 53.5)
- added H3: M2.5, MountingHole:MountingHole_2.7mm_M2.5_Pad, F.Cu at (53.5, 102.5)
- added H4: M2.5, MountingHole:MountingHole_2.7mm_M2.5_Pad, F.Cu at (53.5, 53.5)
- added J1: VBAT, Connector_PinHeader_2.54mm:PinHeader_1x02_P2.54mm_Vertical, F.Cu at (123.7, 102.1)
- added J10: SWD, Connector_PinHeader_2.54mm:PinHeader_1x04_P2.54mm_Horizontal, B.Cu at (83.0, 61.4)
- added J11: BOOT, Connector_PinHeader_2.54mm:PinHeader_1x02_P2.54mm_Horizontal, B.Cu at (90.6, 61.4)
- added J2: VBAT_JST, Connector_JST:JST_PH_S2B-PH-K_1x02_P2.00mm_Horizontal, B.Cu at (122.5, 94.0)
- added J3: USB_C_Receptacle_USB2.0, Connector_USB:USB_C_Receptacle_HRO_TYPE-C-31-M-12, F.Cu at (75.0, 101.0)
- added J4: VIN, libraries:TerminalBlock_KF301-2P, B.Cu at (62.7, 100.8)
- added J5: VOUT, Connector_PinHeader_2.54mm:PinHeader_1x02_P2.54mm_Vertical, F.Cu at (128.7, 55.1)
- added J6: UART1, Connector_PinHeader_2.54mm:PinHeader_1x04_P2.54mm_Vertical, F.Cu at (97.0, 102.1)
- added J7: UART2, Connector_PinHeader_2.54mm:PinHeader_1x04_P2.54mm_Vertical, F.Cu at (97.0, 99.5)
- added J8: Pogo pins, Connector_PinHeader_2.54mm:PinHeader_2x05_P2.54mm_Vertical, F.Cu at (58.4, 54.8)
- added J9: VCC, Connector_PinHeader_2.54mm:PinHeader_1x02_P2.54mm_Vertical, F.Cu at (123.7, 55.1)
- added JP1: S_GND, Jumper:SolderJumper-2_P1.3mm_Open_RoundedPad1.0x1.5mm, F.Cu at (83.0, 102.0)
- added JP2: Cut for 1.5A, Jumper:SolderJumper-2_P1.3mm_Bridged_RoundedPad1.0x1.5mm, F.Cu at (56.5, 71.0)
- added JP4: ADDR, Jumper:SolderJumper-3_P1.3mm_Bridged12_RoundedPad1.0x1.5mm, F.Cu at (96.0, 60.0)
- added L1: 15u 20%, libraries:L_1050, F.Cu at (65.5, 84.5)
- added L2: 1u 20%, libraries:L_7030, F.Cu at (88.0, 79.0)
- added Q3: BATFET, Package_TO_SOT_SMD:SOT-23, F.Cu at (86.0, 111.0)
- added Q4: TDM3412, libraries:DFN3x3E-8_EP2_S, F.Cu at (65.5, 93.0)
- added R1: 20m, Resistor_SMD:R_1206_3216Metric, F.Cu at (91.5, 87.5)
- added R10: 100k, Resistor_SMD:R_0805_2012Metric, F.Cu at (66.0, 73.0)
- added R11: 100k, Resistor_SMD:R_0805_2012Metric, F.Cu at (66.0, 69.5)
- added R12: 100k, Resistor_SMD:R_0805_2012Metric, F.Cu at (62.5, 74.0)
- added R13: 5m 1%, Resistor_SMD:R_1206_3216Metric, F.Cu at (61.0, 61.0)
- added R14: 56k, Resistor_SMD:R_0805_2012Metric, F.Cu at (69.0, 73.0)
- added R15: 4k7, Resistor_SMD:R_0805_2012Metric, F.Cu at (69.0, 69.5)
- added R16: 22k, Resistor_SMD:R_0805_2012Metric, F.Cu at (59.0, 74.0)
- added R17: 18k, Resistor_SMD:R_0805_2012Metric, F.Cu at (59.0, 71.0)
- added R18: R_Small, Resistor_SMD:R_0805_2012Metric, F.Cu at (53.5, 92.0)
- added R19: R_Small, Resistor_SMD:R_0805_2012Metric, F.Cu at (53.5, 88.0)
- added R2: R_Small, Resistor_SMD:R_0805_2012Metric, F.Cu at (27.5, 82.0)
- added R20: R_Small, Resistor_SMD:R_0805_2012Metric, F.Cu at (53.5, 84.0)
- added R21: 100k, Resistor_SMD:R_0805_2012Metric, F.Cu at (16.0, 131.0)
- added R22: R_Small, Resistor_SMD:R_0805_2012Metric, F.Cu at (88.0, 88.0)
- added R23: 100k, Resistor_SMD:R_0805_2012Metric, F.Cu at (16.0, 135.0)
- added R24: R_Small, Resistor_SMD:R_0805_2012Metric, F.Cu at (88.0, 90.0)
- added R25: 10k 1%, Resistor_SMD:R_0805_2012Metric, F.Cu at (82.0, 82.0)
- added R26: 4k7, Resistor_SMD:R_0805_2012Metric, F.Cu at (121.0, 89.0)
- added R27: 4k7, Resistor_SMD:R_0805_2012Metric, F.Cu at (113.0, 82.0)
- added R28: R_Small, Resistor_SMD:R_0805_2012Metric, F.Cu at (126.0, 89.0)
- added R29: R_Small, Resistor_SMD:R_0805_2012Metric, F.Cu at (126.0, 87.0)
- added R3: 5k1, Resistor_SMD:R_0805_2012Metric, F.Cu at (82.0, 97.0)
- added R30: 4k7, Resistor_SMD:R_0805_2012Metric, F.Cu at (121.0, 91.0)
- added R31: 4k7, Resistor_SMD:R_0805_2012Metric, F.Cu at (115.0, 82.0)
- added R32: 402k 1%, Resistor_SMD:R_0805_2012Metric, F.Cu at (75.0, 78.0)
- added R33: R_Small, Resistor_SMD:R_0805_2012Metric, F.Cu at (126.0, 85.0)
- added R34: 8k2 1%, Resistor_SMD:R_0805_2012Metric, F.Cu at (82.0, 84.0)
- added R35: R_Small, Resistor_SMD:R_0805_2012Metric, F.Cu at (73.0, 75.0)
- added R36: 100k 1%, Resistor_SMD:R_0805_2012Metric, F.Cu at (72.0, 78.0)
- added R37: 180R 1%, Resistor_SMD:R_0805_2012Metric, F.Cu at (78.0, 83.0)
- added R38: 0R, Resistor_SMD:R_0805_2012Metric, F.Cu at (95.0, 70.0)
- added R39: 5m 1%, Resistor_SMD:R_1206_3216Metric, F.Cu at (99.0, 69.0)
- added R4: 5k1, Resistor_SMD:R_0805_2012Metric, F.Cu at (85.0, 97.0)
- added R40: 0R, Resistor_SMD:R_0805_2012Metric, F.Cu at (95.0, 68.0)
- added R41: 10k, Resistor_SMD:R_0805_2012Metric, F.Cu at (92.0, 97.0)
- added R42: ??, Resistor_SMD:R_0805_2012Metric, F.Cu at (80.0, 65.0)
- added R43: 10k, Resistor_SMD:R_0805_2012Metric, F.Cu at (78.0, 65.0)
- added R5: R_Small, Resistor_SMD:R_0805_2012Metric, F.Cu at (72.0, 129.0)
- added R6: 10R, Resistor_SMD:R_0805_2012Metric, F.Cu at (60.5, 108.5)
- added R7: 1k, Resistor_SMD:R_0805_2012Metric, F.Cu at (22.5, 82.0)
- added R8: 1k, Resistor_SMD:R_0805_2012Metric, F.Cu at (72.0, 134.0)
- added R9: 20m, Resistor_SMD:R_1206_3216Metric, F.Cu at (63.0, 77.0)
- added SW1: RST, Button_Switch_SMD:SW_Push_1P1T_NO_Vertical_Wuerth_434133025816, F.Cu at (91.0, 102.0)
- added U1: MAX17260SETD+T, Package_DFN_QFN:TDFN-14-1EP_3x3mm_P0.4mm_EP1.78x2.35mm, F.Cu at (61.0, 65.0)
- added U2: BQ24630RGER, libraries:QFN50P400X400X100-25N, F.Cu at (77.0, 89.0)
- added U3: AP22966DC8-7, libraries:V-DFN3020-14, F.Cu at (106.0, 63.0)
- added U4: TPS61230DRC, Package_SON:Texas_S-PVSON-N10_ThermalVias, F.Cu at (79.0, 78.0)
- added U5: STM32F030C8Tx, Package_QFP:LQFP-48_7x7mm_P0.5mm, F.Cu at (110.0, 90.0)
- added U6: INA219AxD, Package_SO:SOIC-8_3.9x4.9mm_P1.27mm, F.Cu at (87.0, 69.0)
- added U7: NCP1117-3.3_SOT223, Package_TO_SOT_SMD:SOT-223-3_TabPin2, F.Cu at (102.0, 79.0)
- added Y1: Crystal_Small, Crystal:Crystal_SMD_HC49-SD, F.Cu at (120.0, 75.0)
Routing:
- net PG: track 0.00 -> 107.3 mm, vias 0 -> 7
- net SDA1: track 0.00 -> 107.3 mm, vias 0 -> 3
- net STAT1: track 0.00 -> 100.6 mm, vias 0 -> 8
- net SDA2: track 0.00 -> 99.5 mm, vias 0 -> 1
- net SCL2: track 0.00 -> 98.2 mm, vias 0 -> 1
- net STAT2: track 0.00 -> 94.9 mm, vias 0 -> 4
- net SCL1: track 0.00 -> 90.0 mm, vias 0 -> 3
- net ALRT: track 0.00 -> 79.6 mm, vias 0 -> 2
- net SWCLK: track 0.00 -> 61.1 mm, vias 0 -> 1
- net SWDIO: track 0.00 -> 58.8 mm, vias 0 -> 1
- net BOOT0: track 0.00 -> 58.7 mm, vias 0 -> 2
- net 5VPG: track 0.00 -> 50.0 mm, vias 0 -> 2
- net CE: track 0.00 -> 45.8 mm, vias 0 -> 6
- net VREF: track 0.00 -> 45.5 mm, vias 0 -> 2
- net Net-(JP2-Pad2): track 0.00 -> 43.4 mm, vias 0 -> 3
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- added copper zone on F.Cu, net +3V3
- added copper zone on In2.Cu, net +3V3
- added copper zone on F.Cu, net +5V
- added copper zone on In2.Cu, net +5V
- added copper zone on F.Cu, net 5VPI
- added copper zone on F.Cu, net 5VPIH
- added copper zone on F.Cu, net BAT
- added copper zone on In2.Cu, net BAT
- added copper zone on F.Cu, net BAT-
- added copper zone on In2.Cu, net BAT-
- added copper zone on B.Cu, net GND
- added copper zone on F.Cu, net GND
- added copper zone on In1.Cu, net GND
- added copper zone on F.Cu, net Net-(C15-Pad2)
- added copper zone on B.Cu, net Net-(J3-PadS1)
- added copper zone on F.Cu, net Net-(J3-PadS1)
- added copper zone on F.Cu, net Net-(L2-Pad2)
- added copper zone on F.Cu, net VBUS
- added copper zone on F.Cu, net VCC
- added copper zone on In2.Cu, net VCC
- added copper zone on F.Cu, net VCCH
Other:
- copper layers 2 -> 4
